Commit message: Add files via upload

File: diffdrive_arduino/description/urdf/diffbot_description.urdf.xacro (robot description, xacro)
@@ -10,5 +10,5 @@
   <xacro:property name="wheel_mass" value="0.3" /> <!-- arbitrary value for wheel mass -->
   <xacro:property name="wheel_len" value="0.050" />
-  <xacro:property name="wheel_radius" value="0.03" />
+  <xacro:property name="wheel_radius" value="0.018" />
   <xacro:property name="caster_wheel_mass" value="0.1" /> <!-- arbitrary value for caster wheel mass -->
   <xacro:property name="caster_wheel_radius" value="0.015" />
